File: Esp32Relays/eagle/neopixel.brd (EAGLE design)
At the start: 54.4 x 16.6 mm, 18 parts, among them J1 Audio2, J3 AUDIO_JACK_3.5MM_PTH, J4 AUDIO_JACK_3.5MM_PTH, U1 CD4066BE

Commit message: Neopixel board
Parts:
- added J2, J5: (no value), SparkFun-Connectors:1X03
- moved R2 4.57 mm to (29.3, 9.65)
- moved R4 4.57 mm to (29.3, 7.05)
- moved C1 4.57 mm to (33.2, 9.65)
- moved C3 4.57 mm to (33.1, 7.05)
- moved R1 4.38 mm to (37.1, 7.11)
- moved R3 4.38 mm to (37.1, 9.72)
- moved R6 0.28 mm to (25.1, 7.05)
- moved C5 0.25 mm to (21.5, 7.05)
- moved R5 0.18 mm to (25.1, 9.59)
- moved C4 0.13 mm to (21.5, 9.59)
Connections:
- net 3V3: now also J2.2, J5.2
- net D25: now also J2.3
- net D26: now also J5.3
- net GND: now also J2.1, J5.1
Routing:
- net D25: track 0.00 -> 26.0 mm
- net 3V3: track 34.3 -> 58.6 mm, vias 2 -> 3
- net B1-SIG-IN: track 30.6 -> 8.62 mm, vias 2 -> 0
- net D26: track 0.00 -> 19.0 mm, vias 0 -> 1
- net VIN: track 48.5 -> 33.1 mm, vias 1 -> 2
- net D12: track 14.9 -> 28.0 mm, vias 0 -> 2
- net A1-SIG-IN: track 24.0 -> 14.8 mm, vias 5 -> 1
- net A2OUT: track 28.6 -> 20.6 mm
- net B2IN: track 20.4 -> 28.0 mm, vias 1 -> 0
- net D27: track 16.4 -> 22.6 mm
- net B1IN: track 24.2 -> 28.7 mm
- net N$2: track 28.1 -> 24.3 mm, vias 4 -> 2
- net D14: track 24.6 -> 21.2 mm, vias 3 -> 0
- net GND: track 95.1 -> 98.4 mm, vias 2 -> 0
- net D13: track 28.6 -> 25.5 mm, vias 2 -> 1
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Other:
- board text added: "5V GND 3.3v"
- board text added: "D25 3.3V G"
- board text added: "D26 3.3V G"
- board text added: "G 3.3V D25"
- board text removed: "5V GND 3v3"

Commit message: Schematic update
Connections:
- net A1-SIG-IN: now also C1.2; no longer C1.1
- net A1-SIG-OUT: now also C4.2, R6.2; no longer C4.1, R5.2
- net A1IN: now also C1.1; no longer C1.2
- net A1OUT: now also C4.1; no longer C4.2
- net B1-SIG-IN: now also C3.2; no longer C3.1
- net B1-SIG-OUT: now also C5.2, R5.2; no longer C5.1, R6.2
- net B1IN: now also C3.1; no longer C3.2
- net B1OUT: now also C5.1; no longer C5.2
Routing:
- net D12: track 28.0 -> 14.4 mm, vias 2 -> 0
- net GND: track 98.4 -> 110.9 mm, vias 0 -> 3
- net B2OUT: track 19.9 -> 31.9 mm, vias 0 -> 1
- net B1-SIG-OUT: track 6.16 -> 16.4 mm
- net B2IN: track 28.0 -> 20.9 mm, vias 0 -> 1
- net D14: track 21.2 -> 15.1 mm
- net VIN: track 33.1 -> 38.2 mm, vias 2 -> 3
- net D13: track 25.5 -> 30.2 mm, vias 1 -> 3
- net D33: track 16.8 -> 21.2 mm, vias 0 -> 2
- net D27: track 22.6 -> 18.5 mm
- net A1OUT: track 15.8 -> 19.3 mm, vias 0 -> 1
- net B1IN: track 28.7 -> 26.1 mm
- net A1IN: track 17.5 -> 15.0 mm, vias 0 -> 1
- net D32: track 18.1 -> 20.2 mm, vias 0 -> 1
- net 3V3: track 58.6 -> 56.8 mm
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