File: Esp32Relays/eagle/neopixel.sch (EAGLE design)
At the start: 18 parts, among them J1 Audio2, J3 AUDIO_JACK_3.5MM_PTH, J4 AUDIO_JACK_3.5MM_PTH, U1 CD4066BE

Commit message: Neopixel board
Parts:
- added J2, J5: (no value), SparkFun-Connectors:CONN_03
Connections:
- net 3V3: now also J2.2, J5.2
- net D25: now also J2.3
- net D26: now also J5.3
- net GND: now also J2.1, J5.1
Changed lines of the file:
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@@
 <part name="R6" library="SparkFun-Resistors" deviceset="0.3OHM" device="-0805-1/8W-1%" value="100k"/>
 <part name="C5" library="SparkFun-Capacitors" deviceset="2.2UF" device="-0805-25V-(+80/-20%)" value="2.2uF"/>
+<part name="J2" library="SparkFun-Connectors" library_urn="urn:adsk.eagle:library:513" deviceset="CONN_03" device="" package3d_urn="urn:adsk.eagle:package:38063/1"/>
+<part name="J5" library="SparkFun-Connectors" library_urn="urn:adsk.eagle:library:513" deviceset="CONN_03" device="" package3d_urn="urn:adsk.eagle:package:38063/1"/>
 </parts>
 <sheets>
@@
 <attribute name="VALUE" x="115.316" y="136.779" size="1.778" layer="96" font="vector" rot="R180"/>
 </instance>
+<instance part="J2" gate="J$1" x="30.48" y="142.24" smashed="yes" rot="R180">
+<attribute name="VALUE" x="33.02" y="149.606" size="1.778" layer="96" font="vector" rot="R180"/>
+<attribute name="NAME" x="33.02" y="136.652" size="1.778" layer="95" font="vector" rot="R180"/>
+</instance>
+<instance part="J5" gate="J$1" x="30.48" y="127" smashed="yes" rot="R180">
+<attribute name="VALUE" x="33.02" y="134.366" size="1.778" layer="96" font="vector" rot="R180"/>
+<attribute name="NAME" x="33.02" y="121.412" size="1.778" layer="95" font="vector" rot="R180"/>
+</instance>
 </instances>
 <busses>
@@
 <label x="127" y="154.94" size="1.778" layer="95" xref="yes"/>
 </segment>
+<segment>
+<pinref part="J2" gate="J$1" pin="1"/>
+<wire x1="22.86" y1="144.78" x2="20.32" y2="144.78" width="0.1524" layer="91"/>
+<label x="20.32" y="144.78" size="1.27" layer="95" rot="R180" xref="yes"/>
+</segment>
+<segment>
+<pinref part="J5" gate="J$1" pin="1"/>
+<wire x1="22.86" y1="129.54" x2="20.32" y2="129.54" width="0.1524" layer="91"/>
+<label x="20.32" y="129.54" size="1.27" layer="95" rot="R180" xref="yes"/>
+</segment>
 </net>
 <net name="D13" class="0">
@@
 <label x="66.04" y="73.66" size="1.27" layer="95" xref="yes"/>
 </segment>
+<segment>
+<pinref part="J5" gate="J$1" pin="3"/>
+<wire x1="22.86" y1="124.46" x2="20.32" y2="124.46" width="0.1524" layer="91"/>
+<label x="20.32" y="124.46" size="1.27" layer="95" rot="R180" xref="yes"/>
+</segment>
 </net>
 <net name="D25" class="0">
@@
 <label x="66.04" y="71.12" size="1.27" layer="95" xref="yes"/>
 </segment>
+<segment>
+<pinref part="J2" gate="J$1" pin="3"/>
+<wire x1="22.86" y1="139.7" x2="20.32" y2="139.7" width="0.1524" layer="91"/>
+<label x="20.32" y="139.7" size="1.27" layer="95" rot="R180" xref="yes"/>
+</segment>
 </net>
 <net name="D33" class="0">
@@
 <wire x1="38.1" y1="154.94" x2="33.02" y2="154.94" width="0.1524" layer="91"/>
 <label x="33.02" y="154.94" size="1.778" layer="95" rot="R180" xref="yes"/>
+</segment>
+<segment>
+<pinref part="J2" gate="J$1" pin="2"/>
+<wire x1="22.86" y1="142.24" x2="20.32" y2="142.24" width="0.1524" layer="91"/>
+<label x="20.32" y="142.24" size="1.27" layer="95" rot="R180" xref="yes"/>
+</segment>
+<segment>
+<pinref part="J5" gate="J$1" pin="2"/>
+<wire x1="22.86" y1="127" x2="20.32" y2="127" width="0.1524" layer="91"/>
+<label x="20.32" y="127" size="1.27" layer="95" rot="R180" xref="yes"/>
 </segment>
 </net>
@@
 <pinref part="C1" gate="G$1" pin="1"/>
 <wire x1="66.04" y1="147.32" x2="68.58" y2="147.32" width="0.1524" layer="91"/>
-<wire x1="68.58" y1="147.32" x2="71.12" y2="142.24" width="0.1524" layer="91"/>
+<wire x1="68.58" y1="147.32" x2="68.58" y2="142.24" width="0.1524" layer="91"/>
 <junction x="68.58" y="147.32"/>
-<label x="71.12" y="142.24" size="1.778" layer="95" xref="yes"/>
+<label x="68.58" y="142.24" size="1.27" layer="95" xref="yes"/>
+<wire x1="71.12" y1="142.24" x2="68.58" y2="142.24" width="0.1524" layer="91"/>
 </segment>
 <segment>
@@
 <wire x1="68.58" y1="134.62" x2="71.12" y2="129.54" width="0.1524" layer="91"/>
 <junction x="68.58" y="134.62"/>
-<label x="71.12" y="129.54" size="1.778" layer="95" xref="yes"/>
+<label x="71.12" y="129.54" size="1.27" layer="95" xref="yes"/>
 </segment>
 <segment>
@@
 <wire x1="104.14" y1="147.32" x2="106.68" y2="142.24" width="0.1524" layer="91"/>
 <junction x="104.14" y="147.32"/>
-<label x="106.68" y="142.24" size="1.778" layer="95" xref="yes"/>
+<label x="106.68" y="142.24" size="1.27" layer="95" xref="yes"/>
 </segment>
 </net>
@@
 <wire x1="104.14" y1="134.62" x2="106.68" y2="129.54" width="0.1524" layer="91"/>
 <junction x="104.14" y="134.62"/>
-<label x="106.68" y="129.54" size="1.778" layer="95" xref="yes"/>
-</segment>
-</net>
+<label x="106.68" y="129.54" size="1.27" layer="95" xref="yes"/>
+</segment>
+</net>

Commit message: Schematic update
Connections:
- net A1-SIG-IN: now also C1.2; no longer C1.1
- net A1-SIG-OUT: now also C4.2, R6.2; no longer C4.1, R5.2
- net A1IN: now also C1.1; no longer C1.2
- net A1OUT: now also C4.1; no longer C4.2
- net B1-SIG-IN: now also C3.2; no longer C3.1
- net B1-SIG-OUT: now also C5.2, R5.2; no longer C5.1, R6.2
- net B1IN: now also C3.1; no longer C3.2
- net B1OUT: now also C5.1; no longer C5.2
Other:
- moved on the sheet: C1, C3, C4, C5, DISPLAY, ESP32-RIGHT, J1, J2, J3, J4, J5, POWER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
