File: Lcd3.5Connectors/eagle/Lcd3_5Connect.sch (EAGLE design)
At the start: 4 parts

Commit message: Added 3v3 / GND connection
Parts:
- added JP3: (no value), pinhead:PINHD-1X2
Connections:
- net 3V3: now also JP3.1
- net GND: now also JP3.2
Changed lines of the file:
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@@
 <part name="JP1" library="con-JST XH" deviceset="S4B-XH" device="-A-1"/>
 <part name="JP2" library="pinhead" library_urn="urn:adsk.eagle:library:325" deviceset="PINHD-1X4" device="" package3d_urn="urn:adsk.eagle:package:22407/2"/>
+<part name="JP3" library="pinhead" library_urn="urn:adsk.eagle:library:325" deviceset="PINHD-1X2" device="" package3d_urn="urn:adsk.eagle:package:22435/2"/>
 </parts>
 <sheets>
@@
 <attribute name="VALUE" x="-6.35" y="20.32" size="1.778" layer="96"/>
 </instance>
+<instance part="JP3" gate="G$1" x="58.42" y="33.02" smashed="yes">
+<attribute name="NAME" x="52.07" y="38.735" size="1.778" layer="95"/>
+<attribute name="VALUE" x="52.07" y="27.94" size="1.778" layer="96"/>
+</instance>
 </instances>
 <busses>
@@
 <label x="30.48" y="60.96" size="1.27" layer="95" rot="R180" xref="yes"/>
 </segment>
+<segment>
+<pinref part="JP3" gate="G$1" pin="1"/>
+<wire x1="55.88" y1="35.56" x2="50.8" y2="35.56" width="0.1524" layer="91"/>
+<label x="50.8" y="35.56" size="1.27" layer="95" rot="R180" xref="yes"/>
+</segment>
 </net>
 <net name="GND" class="0">
@@
 <label x="-10.16" y="30.48" size="1.27" layer="95" rot="R180" xref="yes"/>
 </segment>
+<segment>
+<pinref part="JP3" gate="G$1" pin="2"/>
+<wire x1="55.88" y1="33.02" x2="50.8" y2="33.02" width="0.1524" layer="91"/>
+<label x="50.8" y="33.02" size="1.27" layer="95" rot="R180" xref="yes"/>
+</segment>
 </net>

Commit message: Corrected left vs right nomenclature
Parts:
- renumbered ESP32-LEFT to ESP32-RIGHT
Changed lines of the file:
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@@
 </classes>
 <parts>
-<part name="ESP32-LEFT" library="pinhead" library_urn="urn:adsk.eagle:library:325" deviceset="PINHD-1X15" device="" package3d_urn="urn:adsk.eagle:package:22424/2" value="0"/>
+<part name="ESP32-RIGHT" library="pinhead" library_urn="urn:adsk.eagle:library:325" deviceset="PINHD-1X15" device="" package3d_urn="urn:adsk.eagle:package:22424/2" value="0"/>
 <part name="LCD-3.5" library="pinhead" library_urn="urn:adsk.eagle:library:325" deviceset="PINHD-1X14" device="" package3d_urn="urn:adsk.eagle:package:22417/2" value="0"/>
 <part name="JP1" library="con-JST XH" deviceset="S4B-XH" device="-A-1"/>
@@
 </plain>
 <instances>
-<instance part="ESP32-LEFT" gate="A" x="0" y="60.96" smashed="yes">
+<instance part="ESP32-RIGHT" gate="A" x="0" y="60.96" smashed="yes">
 <attribute name="NAME" x="-6.35" y="81.915" size="1.778" layer="95"/>
 <attribute name="VALUE" x="-6.35" y="38.1" size="1.778" layer="96"/>
@@
 <net name="3V3" class="0">
 <segment>
-<pinref part="ESP32-LEFT" gate="A" pin="1"/>
+<pinref part="ESP32-RIGHT" gate="A" pin="1"/>
 <wire x1="-2.54" y1="78.74" x2="-12.7" y2="78.74" width="0.1524" layer="91"/>
 <label x="-12.7" y="78.74" size="1.27" layer="95" rot="R180" xref="yes"/>
@@
 <net name="GND" class="0">
 <segment>
-<pinref part="ESP32-LEFT" gate="A" pin="2"/>
+<pinref part="ESP32-RIGHT" gate="A" pin="2"/>
 <wire x1="-2.54" y1="76.2" x2="-12.7" y2="76.2" width="0.1524" layer="91"/>
 <label x="-12.7" y="76.2" size="1.27" layer="95" rot="R180" xref="yes"/>
@@
 <net name="15" class="0">
 <segment>
-<pinref part="ESP32-LEFT" gate="A" pin="3"/>
+<pinref part="ESP32-RIGHT" gate="A" pin="3"/>
 <wire x1="-2.54" y1="73.66" x2="-12.7" y2="73.66" width="0.1524" layer="91"/>
 <label x="-12.7" y="73.66" size="1.27" layer="95" rot="R180" xref="yes"/>
@@
 <net name="2" class="0">
 <segment>
-<pinref part="ESP32-LEFT" gate="A" pin="4"/>
+<pinref part="ESP32-RIGHT" gate="A" pin="4"/>
 <wire x1="-2.54" y1="71.12" x2="-12.7" y2="71.12" width="0.1524" layer="91"/>
 <label x="-12.7" y="71.12" size="1.27" layer="95" rot="R180" xref="yes"/>
@@
 <net name="4" class="0">
 <segment>
-<pinref part="ESP32-LEFT" gate="A" pin="5"/>
+<pinref part="ESP32-RIGHT" gate="A" pin="5"/>
 <wire x1="-2.54" y1="68.58" x2="-12.7" y2="68.58" width="0.1524" layer="91"/>
 <label x="-12.7" y="68.58" size="1.27" layer="95" rot="R180" xref="yes"/>
@@
 <net name="16" class="0">
 <segment>
-<pinref part="ESP32-LEFT" gate="A" pin="6"/>
+<pinref part="ESP32-RIGHT" gate="A" pin="6"/>
 <wire x1="-2.54" y1="66.04" x2="-12.7" y2="66.04" width="0.1524" layer="91"/>
 <label x="-12.7" y="66.04" size="1.27" layer="95" rot="R180" xref="yes"/>
@@
 <net name="17" class="0">
 <segment>
-<pinref part="ESP32-LEFT" gate="A" pin="7"/>
+<pinref part="ESP32-RIGHT" gate="A" pin="7"/>
 <wire x1="-2.54" y1="63.5" x2="-12.7" y2="63.5" width="0.1524" layer="91"/>
 <label x="-12.7" y="63.5" size="1.27" layer="95" rot="R180" xref="yes"/>
@@
 <net name="5" class="0">
 <segment>
-<pinref part="ESP32-LEFT" gate="A" pin="8"/>
+<pinref part="ESP32-RIGHT" gate="A" pin="8"/>
 <wire x1="-2.54" y1="60.96" x2="-12.7" y2="60.96" width="0.1524" layer="91"/>
 <label x="-12.7" y="60.96" size="1.27" layer="95" rot="R180" xref="yes"/>
@@
 <net name="18" class="0">
 <segment>
-<pinref part="ESP32-LEFT" gate="A" pin="9"/>
+<pinref part="ESP32-RIGHT" gate="A" pin="9"/>
 <wire x1="-2.54" y1="58.42" x2="-12.7" y2="58.42" width="0.1524" layer="91"/>
 <label x="-12.7" y="58.42" size="1.27" layer="95" rot="R180" xref="yes"/>
@@
 <net name="19" class="0">
 <segment>
-<pinref part="ESP32-LEFT" gate="A" pin="10"/>
+<pinref part="ESP32-RIGHT" gate="A" pin="10"/>
 <wire x1="-2.54" y1="55.88" x2="-12.7" y2="55.88" width="0.1524" layer="91"/>
 <label x="-12.7" y="55.88" size="1.27" layer="95" rot="R180" xref="yes"/>
@@
 <net name="21" class="0">
 <segment>
-<pinref part="ESP32-LEFT" gate="A" pin="11"/>
+<pinref part="ESP32-RIGHT" gate="A" pin="11"/>
 <wire x1="-2.54" y1="53.34" x2="-12.7" y2="53.34" width="0.1524" layer="91"/>
 <label x="-12.7" y="53.34" size="1.27" layer="95" rot="R180" xref="yes"/>
@@
 <net name="22" class="0">
 <segment>
-<pinref part="ESP32-LEFT" gate="A" pin="14"/>
+<pinref part="ESP32-RIGHT" gate="A" pin="14"/>
 <wire x1="-2.54" y1="45.72" x2="-12.7" y2="45.72" width="0.1524" layer="91"/>
 <label x="-12.7" y="45.72" size="1.27" layer="95" rot="R180" xref="yes"/>
@@
 <net name="23" class="0">
 <segment>
-<pinref part="ESP32-LEFT" gate="A" pin="15"/>
+<pinref part="ESP32-RIGHT" gate="A" pin="15"/>
 <wire x1="-2.54" y1="43.18" x2="-12.7" y2="43.18" width="0.1524" layer="91"/>
 <label x="-12.7" y="43.18" size="1.27" layer="95" rot="R180" xref="yes"/>

Commit message: Added brightness GPIO
and removed - unused - Touch IRQ pin
Connections:
- net 15: now also LCD-3.5.8; no longer LCD-3.5.14
- net 3V3: no longer LCD-3.5.8
Changed lines of the file:
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@@
-</segment>
-<segment>
-<pinref part="LCD-3.5" gate="A" pin="8"/>
-<wire x1="40.64" y1="60.96" x2="30.48" y2="60.96" width="0.1524" layer="91"/>
-<label x="30.48" y="60.96" size="1.27" layer="95" rot="R180" xref="yes"/>
 </segment>
 <segment>
@@
 </segment>
 <segment>
-<pinref part="LCD-3.5" gate="A" pin="14"/>
-<wire x1="40.64" y1="45.72" x2="30.48" y2="45.72" width="0.1524" layer="91"/>
-<label x="30.48" y="45.72" size="1.27" layer="95" rot="R180" xref="yes"/>
+<pinref part="LCD-3.5" gate="A" pin="8"/>
+<wire x1="40.64" y1="60.96" x2="30.48" y2="60.96" width="0.1524" layer="91"/>
+<label x="30.48" y="60.96" size="1.27" layer="95" rot="R180" xref="yes"/>
 </segment>
 </net>

Commit message: Work on scad output
Parts:
- JP3: device pinhead:PINHD-1X2 -> SparkFun-Connectors:CONN_02
Other:
- moved on the sheet: JP3
Changed lines of the file:
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@@
 <layer number="48" name="Document" color="7" fill="1" visible="no" active="no"/>
 <layer number="49" name="Reference" color="7" fill="1" visible="no" active="no"/>
+<layer number="50" name="dxf" color="7" fill="1" visible="no" active="no"/>
 <layer number="51" name="tDocu" color="7" fill="1" visible="no" active="no"/>
 <layer number="52" name="bDocu" color="7" fill="1" visible="no" active="no"/>
+<layer number="53" name="tGND_GNDA" color="7" fill="9" visible="no" active="no"/>
+<layer number="54" name="bGND_GNDA" color="1" fill="9" visible="no" active="no"/>
+<layer number="56" name="wert" color="7" fill="1" visible="no" active="no"/>
+<layer number="57" name="tCAD" color="7" fill="1" visible="no" active="no"/>
+<layer number="59" name="tCarbon" color="7" fill="1" visible="no" active="no"/>
+<layer number="60" name="bCarbon" color="7" fill="1" visible="no" active="no"/>
 <layer number="88" name="SimResults" color="9" fill="1" visible="yes" active="yes"/>
 <layer number="89" name="SimProbes" color="9" fill="1" visible="yes" active="yes"/>
@@
 <layer number="97" name="Info" color="7" fill="1" visible="yes" active="yes"/>
 <layer number="98" name="Guide" color="6" fill="1" visible="yes" active="yes"/>
+<layer number="99" name="SpiceOrder" color="7" fill="1" visible="yes" active="yes"/>
+<layer number="100" name="Muster" color="7" fill="1" visible="no" active="no"/>
+<layer number="101" name="Patch_Top" color="12" fill="4" visible="yes" active="yes"/>
+<layer number="102" name="Vscore" color="7" fill="1" visible="yes" active="yes"/>
+<layer number="103" name="tMap" color="7" fill="1" visible="yes" active="yes"/>
+<layer number="104" name="Name" color="16" fill="1" visible="yes" active="yes"/>
+<layer number="105" name="tPlate" color="7" fill="1" visible="yes" active="yes"/>
+<layer number="106" name="bPlate" color="7" fill="1" visible="yes" active="yes"/>
+<layer number="107" name="Crop" color="7" fill="1" visible="yes" active="yes"/>
+<layer number="108" name="tplace-old" color="10" fill="1" visible="yes" active="yes"/>
+<layer number="109" name="ref-old" color="11" fill="1" visible="yes" active="yes"/>
+<layer number="110" name="fp0" color="7" fill="1" visible="yes" active="yes"/>
+<layer number="111" name="LPC17xx" color="7" fill="1" visible="yes" active="yes"/>
+<layer number="112" name="tSilk" color="7" fill="1" visible="yes" active="yes"/>
+<layer number="113" name="IDFDebug" color="4" fill="1" visible="yes" active="yes"/>
+<layer number="114" name="Badge_Outline" color="7" fill="1" visible="yes" active="yes"/>
+<layer number="115" name="ReferenceISLANDS" color="7" fill="1" visible="yes" active="yes"/>
+<layer number="116" name="Patch_BOT" color="9" fill="4" visible="yes" active="yes"/>
+<layer number="118" name="Rect_Pads" color="7" fill="1" visible="yes" active="yes"/>
+<layer number="121" name="_tsilk" color="7" fill="1" visible="yes" active="yes"/>
+<layer number="122" name="_bsilk" color="7" fill="1" visible="yes" active="yes"/>
+<layer number="123" name="tTestmark" color="7" fill="1" visible="yes" active="yes"/>
+<layer number="124" name="bTestmark" color="7" fill="1" visible="yes" active="yes"/>
+<layer number="125" name="_tNames" color="7" fill="1" visible="yes" active="yes"/>
+<layer number="126" name="_bNames" color="7" fill="1" visible="yes" active="yes"/>
+<layer number="127" name="_tValues" color="7" fill="1" visible="yes" active="yes"/>
+<layer number="128" name="_bValues" color="7" fill="1" visible="yes" active="yes"/>
+<layer number="129" name="Mask" color="7" fill="1" visible="yes" active="yes"/>
+<layer number="131" name="tAdjust" color="7" fill="1" visible="yes" active="yes"/>
+<layer number="132" name="bAdjust" color="7" fill="1" visible="yes" active="yes"/>
+<layer number="144" name="Drill_legend" color="7" fill="1" visible="yes" active="yes"/>
+<layer number="150" name="Notes" color="7" fill="1" visible="yes" active="yes"/>
+<layer number="151" name="HeatSink" color="7" fill="1" visible="yes" active="yes"/>
+<layer number="152" name="_bDocu" color="7" fill="1" visible="yes" active="yes"/>
+<layer number="153" name="FabDoc1" color="7" fill="1" visible="yes" active="yes"/>
+<layer number="154" name="FabDoc2" color="7" fill="1" visible="yes" active="yes"/>
+<layer number="155" name="FabDoc3" color="7" fill="1" visible="yes" active="yes"/>
+<layer number="199" name="Contour" color="7" fill="1" visible="yes" active="yes"/>
+<layer number="200" name="200bmp" color="1" fill="10" visible="yes" active="yes"/>
+<layer number="201" name="201bmp" color="2" fill="10" visible="yes" active="yes"/>
+<layer number="202" name="202bmp" color="3" fill="10" visible="yes" active="yes"/>
+<layer number="203" name="203bmp" color="4" fill="10" visible="yes" active="yes"/>
+<layer number="204" name="204bmp" color="5" fill="10" visible="yes" active="yes"/>
+<layer number="205" name="205bmp" color="6" fill="10" visible="yes" active="yes"/>
+<layer number="206" name="206bmp" color="7" fill="10" visible="yes" active="yes"/>
+<layer number="207" name="207bmp" color="8" fill="10" visible="yes" active="yes"/>
+<layer number="208" name="208bmp" color="9" fill="10" visible="yes" active="yes"/>
+<layer number="209" name="209bmp" color="7" fill="1" visible="yes" active="yes"/>
+<layer number="210" name="210bmp" color="7" fill="1" visible="yes" active="yes"/>
+<layer number="211" name="211bmp" color="7" fill="1" visible="yes" active="yes"/>
+<layer number="212" name="212bmp" color="7" fill="1" visible="yes" active="yes"/>
+<layer number="213" name="213bmp" color="7" fill="1" visible="yes" active="yes"/>
+<layer number="214" name="214bmp" color="7" fill="1" visible="yes" active="yes"/>
+<layer number="215" name="215bmp" color="7" fill="1" visible="yes" active="yes"/>
+<layer number="216" name="216bmp" color="7" fill="1" visible="yes" active="yes"/>
+<layer number="217" name="217bmp" color="18" fill="1" visible="no" active="no"/>
+<layer number="218" name="218bmp" color="19" fill="1" visible="no" active="no"/>
+<layer number="219" name="219bmp" color="20" fill="1" visible="no" active="no"/>
+<layer number="220" name="220bmp" color="21" fill="1" visible="no" active="no"/>
+<layer number="221" name="221bmp" color="22" fill="1" visible="no" active="no"/>
+<layer number="222" name="222bmp" color="23" fill="1" visible="no" active="no"/>
+<layer number="223" name="223bmp" color="24" fill="1" visible="no" active="no"/>
+<layer number="224" name="224bmp" color="25" fill="1" visible="no" active="no"/>
+<layer number="225" name="225bmp" color="7" fill="1" visible="yes" active="yes"/>
+<layer number="226" name="226bmp" color="7" fill="1" visible="yes" active="yes"/>
+<layer number="227" name="227bmp" color="7" fill="1" visible="yes" active="yes"/>
+<layer number="228" name="228bmp" color="7" fill="1" visible="yes" active="yes"/>
+<layer number="229" name="229bmp" color="7" fill="1" visible="yes" active="yes"/>
+<layer number="230" name="230bmp" color="7" fill="1" visible="yes" active="yes"/>
+<layer number="231" name="231bmp" color="7" fill="1" visible="yes" active="yes"/>
+<layer number="232" name="Eagle3D_PG2" color="7" fill="1" visible="yes" active="yes"/>
+<layer number="233" name="Eagle3D_PG3" color="7" fill="1" visible="yes" active="yes"/>
+<layer number="248" name="Housing" color="7" fill="1" visible="yes" active="yes"/>
+<layer number="249" name="Edge" color="7" fill="1" visible="yes" active="yes"/>
+<layer number="250" name="Descript" color="3" fill="1" visible="no" active="no"/>
+<layer number="251" name="SMDround" color="12" fill="11" visible="no" active="no"/>
+<layer number="254" name="cooling" color="7" fill="1" visible="yes" active="yes"/>
+<layer number="255" name="routoute" color="7" fill="1" visible="yes" active="yes"/>
 </layers>
 <schematic xreflabel="%F%N/%S.%C%R" xrefpart="/%S.%C%R">
@@
 <part name="JP1" library="con-JST XH" deviceset="S4B-XH" device="-A-1"/>
 <part name="JP2" library="pinhead" library_urn="urn:adsk.eagle:library:325" deviceset="PINHD-1X4" device="" package3d_urn="urn:adsk.eagle:package:22407/2"/>
-<part name="JP3" library="pinhead" library_urn="urn:adsk.eagle:library:325" deviceset="PINHD-1X2" device="" package3d_urn="urn:adsk.eagle:package:22435/2"/>
+<part name="JP3" library="SparkFun-Connectors" library_urn="urn:adsk.eagle:library:513" deviceset="CONN_02" device="" package3d_urn="urn:adsk.eagle:package:38039/1"/>
 </parts>
 <sheets>
@@
 <attribute name="VALUE" x="-6.35" y="20.32" size="1.778" layer="96"/>
 </instance>
-<instance part="JP3" gate="G$1" x="58.42" y="33.02" smashed="yes">
-<attribute name="NAME" x="52.07" y="38.735" size="1.778" layer="95"/>
-<attribute name="VALUE" x="52.07" y="27.94" size="1.778" layer="96"/>
+<instance part="JP3" gate="G$1" x="60.96" y="35.56" smashed="yes" rot="R180">
+<attribute name="NAME" x="67.31" y="29.845" size="1.778" layer="95" rot="R180"/>
+<attribute name="VALUE" x="67.31" y="40.64" size="1.778" layer="96" rot="R180"/>
 </instance>
 </instances>
@@
 <segment>
 <pinref part="JP3" gate="G$1" pin="1"/>
-<wire x1="55.88" y1="35.56" x2="50.8" y2="35.56" width="0.1524" layer="91"/>
+<wire x1="53.34" y1="35.56" x2="50.8" y2="35.56" width="0.1524" layer="91"/>
 <label x="50.8" y="35.56" size="1.27" layer="95" rot="R180" xref="yes"/>
 </segment>
@@
 <segment>
 <pinref part="JP3" gate="G$1" pin="2"/>
-<wire x1="55.88" y1="33.02" x2="50.8" y2="33.02" width="0.1524" layer="91"/>
+<wire x1="53.34" y1="33.02" x2="50.8" y2="33.02" width="0.1524" layer="91"/>
 <label x="50.8" y="33.02" size="1.27" layer="95" rot="R180" xref="yes"/>
 </segment>
